File: hardware/orrery_v1/orrery_v1.kicad_sch (KiCad schematic)
At the start: 0 parts

Commit message: hardware: complete orrery_v1 schematic
Full ESP32-S3 + HUB75 + peripherals wired up. Netlist verified
against firmware/main/pins.h — all GPIO assignments match.

Highlights:
- U1 ESP32-S3-DevKitC driving HUB75 J2 (2x8 IDC), pin-perfect map to
  R1/G1/B1/R2/G2/B2/A-D/CLK/LAT/OE per pins.h
- J2 pin 8 (E) grounded via R1 0-ohm jumper (upgrade path to 1:32
  scan panels later)
- U2 BH1750 on I2C bus (GPIO 41/42), ADDR tied to GND for 0x23
- SW1 KY-040 encoder on GPIO 38/39/40, C4 debounce on SW
- U3 MAX98357A on I2S (GPIO 9/10/11), GAIN and SD left floating
  (9 dB, mono mix); C2/C3 local decoupling on VIN
- LS1 speaker documented as board-external; J5 JST-PH 2P on the main
  PCB provides the mechanical anchor for the pigtail
- J1 5V power in from external RS-25-5, J4 dedicated 5V feed to
  HUB75 panel power lugs
- C1 1000 uF bulk on 5V rail; C5/C6, C7/C8 additional decoupling
- All PSRAM range (GPIO 26-37) and USB/UART pins left no_connect;
  strapping pins (0, 3, 45, 46) and free GPIOs (1, 8, 12, 13) also
  NC-flagged
- AC entirely off the PCB: C14 inlet and RS-25-5 PSU are chassis-
  mount, hand-wired to J1 screw terminal

Co-Authored-By: Claude Opus 4.7 <noreply@anthropic.com>
Parts:
- added C1, C2: 1000uF, 25V, Capacitor_THT:CP_Radial_D10.0mm_P5.00mm, symbol Device:C_Polarized
- added C3, C4, C6, C7: 100nF, 100V, Capacitor_THT:C_Disc_D10.0mm_W2.5mm_P5.00mm, symbol Device:C
- added C5, C8: 100uF, 25V, Capacitor_THT:CP_Radial_D10.0mm_P5.00mm, symbol Device:C_Polarized
- added H1, H10, H11, H12, H2, H3, H4, H5, H6, H7, H8, H9: MountingHole, MountingHole:MountingHole_3.2mm_M3_ISO7380, symbol Mechanical:MountingHole
- added J1, J4: Screw_Terminal_01x02, TerminalBlock_Phoenix:TerminalBlock_Phoenix_MKDS-1,5-2-5.08_1x02_P5.08mm_Horizontal, symbol Connector:Screw_Terminal_01x02
- added J2: Conn_02x08_Odd_Even, Connector_IDC:IDC-Header_2x08_P2.54mm_Vertical, symbol Connector_Generic:Conn_02x08_Odd_Even
- added J3: IEC_60320_C14_Receptacle, symbol Connector:IEC_60320_C14_Receptacle
- added LS1: Speaker 3W 8Ohm, TerminalBlock_Phoenix:TerminalBlock_Phoenix_MKDS-1,5-2-5.08_1x02_P5.08mm_Horizontal, symbol Orrery:Speaker_3W_8Ohm
- added P1: Conn_Plug_3P_Protected, symbol Connector:Conn_Plug_3P_Protected
- added P2: IEC_60320_C13_Plug, symbol Connector:IEC_60320_C13_Plug
- added PS1: RS-25-5, symbol Orrery:RS-25-5
- added R1: 0, Resistor_THT:R_Axial_DIN0207_L6.3mm_D2.5mm_P10.16mm_Horizontal, symbol Device:R
- added SW1: KY-040, Connector_PinHeader_2.54mm:PinHeader_1x05_P2.54mm_Vertical, symbol Orrery:KY-040
- added U1: ESP32-S3-DevKitC, Espressif:ESP32-S3-DevKitC, symbol Espressif:ESP32-S3-DevKitC
- added U2: BH1750_GY-302, Connector_PinHeader_2.54mm:PinHeader_1x05_P2.54mm_Vertical, symbol Orrery:BH1750_GY-302
- added U3: MAX98357A, Connector_PinHeader_2.54mm:PinHeader_1x07_P2.54mm_Vertical, symbol Orrery:MAX98357A
Connections:
- new net: J2.8 (Pin_8), R1.2
- new net: J3.1 (L), PS1.5 (AC/L)
- new net: J3.2 (N), PS1.4 (AC/N)
- new net: J3.3 (PE), PS1.6 (PE)
- new net: LS1.1 (+), U3.8 (OUT+)
- new net: LS1.2 (-), U3.9 (OUT-)
- new net: P1.2 (N), P2.1 (N)
- new net: P1.1 (L), P2.2 (L)
- new net: P1.3 (PE), P2.3 (PE)
- new net +3V3: C7.1, C8.1, SW1.4 (+), U1.1 (3V3), U1.2 (3V3), U2.1 (VCC)
- new net +5V: C1.1, C2.1, C3.1, C5.1, C6.1, J1.1 (Pin_1), J4.1 (Pin_1), PS1.2 (+V), U1.21 (5V), U3.6 (VIN)
- new net BH1750_SCL: U1.39 (GPIO42/MTMS), U2.3 (SCL)
- new net BH1750_SDA: U1.38 (GPIO41/MTDI), U2.4 (SDA)
- new net GND: C1.2, C2.2, C3.2, C4.2, C5.2, C6.2, C7.2, C8.2, J1.2 (Pin_2), J2.16 (Pin_16), J2.4 (Pin_4), J4.2 (Pin_2), PS1.1 (-V), R1.1, SW1.5 (GND), U1.22 (GND), U1.23 (GND), U1.24 (GND), U1.44 (GND), U2.2 (GND), U2.5 (ADDR), U3.7 (GND)
- new net HUB75_A: J2.9 (Pin_9), U1.10 (GPIO17/ADC2_CH6)
- new net HUB75_B: J2.10 (Pin_10), U1.11 (GPIO18/ADC2_CH7)
- new net HUB75_B1: J2.3 (Pin_3), U1.6 (GPIO6/ADC1_CH5)
- new net HUB75_B2: J2.7 (Pin_7), U1.9 (GPIO16/ADC2_CH5/32K_N)
- new net HUB75_C: J2.11 (Pin_11), U1.27 (GPIO21)
- new net HUB75_CLK: J2.13 (Pin_13), U1.40 (GPIO2/ADC1_CH1)
- new net HUB75_D: J2.12 (Pin_12), U1.20 (GPIO14/ADC2_CH3)
- new net HUB75_G1: J2.2 (Pin_2), U1.5 (GPIO5/ADC1_CH4)
- new net HUB75_G2: J2.6 (Pin_6), U1.8 (GPIO15/ADC2_CH4/32K_P)
- new net HUB75_LAT: J2.14 (Pin_14), U1.28 (GPIO47)
- new net HUB75_OE: J2.15 (Pin_15), U1.29 (GPIO48)
- new net HUB75_R1: J2.1 (Pin_1), U1.4 (GPIO4/ADC1_CH3)
- new net HUB75_R2: J2.5 (Pin_5), U1.7 (GPIO7/ADC1_CH6)
- new net KY-040_CLK: SW1.1 (CLK), U1.37 (GPIO40/MTDO)
- new net KY-040_DT: SW1.2 (DT), U1.36 (GPIO39/MTCK)
- new net KY-040_SW: C4.1, SW1.3 (SW), U1.35 (GPIO38)
- new net MAX98357A_BCLK: U1.15 (GPIO9/ADC1_CH8), U3.2 (BCLK)
- new net MAX98357A_DIN: U1.17 (GPIO11/ADC2_CH0), U3.3 (DIN)
- new net MAX98357A_LRC: U1.16 (GPIO10/ADC1_CH9), U3.1 (LRC)
- no-connect marks 0 -> 18
Other:
- note added: "5V Power Supply Input to Board"
- note added: "5V Power Supply Output to HUB75"
- note added: "Connector to HUB75 LED Matrix"
- note added: "Display: - LED Matrix HUB 75 32x64 Microcontroller: - ESP-S3-DevKitC-1 Audio: - MAX98357A I2S 3W Mono Amplifier Class D Filterless Amplifier Breakout Module - GERUI DFplayer Mini 3 Watt 8 Ohm Speaker with JST-PH2.0 mm Pin Light Sensor - GY-302 BH1750 BH1750FVI Rotary Encoder - Taiss Rotary Encoder Module KY-040 360 Power Supply: - Rectifier 5V, 5A, Meanwell RS-25-5 - Cable: IEC C13 Power Cord wit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"
- note added: "IEC 60320 C14 panel-mount inlet with integrated rocker switch and fuse holder"
- note added: "IEC C13 Power Cord with CEE 7/7 (Schuko) Plug"
- note added: "MeanWell Power Supply Mounting Holes"
- note added: "PCB-to-HUB75 Mounting Holes"
- note added: "Power supply not part of the PCB but mounted in the PCB."
- note added: "Speaker Mounting Holes"

Commit message: hardware: iterate on orrery_v1 PCB layout + refresh STEP
Continues the board bring-up: schematic tweaks, routing, and zone
settings adjusted. Notable changes visible in the project file:
- Added JP1 to the designator list (E-line jumper as a 2-pad test
  point, per earlier discussion)
- Zone rules: remove_islands enabled, min_clearance dropped to 0
- Component count now up to R1-3 and C1-8

Regenerates mechanical/orrery_v1_pcb.step so the FreeCAD assembly
picks up the same geometry.

Co-Authored-By: Claude Opus 4.7 <noreply@anthropic.com>
Parts:
- removed H10, H11, H12, H5, H6, H7, H8, H9: MountingHole, MountingHole:MountingHole_3.2mm_M3_ISO7380, symbol Mechanical:MountingHole
- removed R1: 0, Resistor_THT:R_Axial_DIN0207_L6.3mm_D2.5mm_P10.16mm_Horizontal, symbol Device:R
- added JP1: Jumper_2_Bridged, TestPoint:TestPoint_2Pads_Pitch2.54mm_Drill0.8mm, symbol Jumper:Jumper_2_Bridged
- C2: value 1000uF, 25V -> 100uF, 25V; footprint Capacitor_THT:CP_Radial_D10.0mm_P5.00mm -> Capacitor_THT:CP_Radial_D5.0mm_P2.50mm
- C3, C4, C6, C7: footprint Capacitor_THT:C_Disc_D10.0mm_W2.5mm_P5.00mm -> Capacitor_THT:C_Disc_D5.0mm_W2.5mm_P2.50mm
- C5, C8: footprint Capacitor_THT:CP_Radial_D10.0mm_P5.00mm -> Capacitor_THT:CP_Radial_D5.0mm_P2.50mm
- U1: footprint Espressif:ESP32-S3-DevKitC -> PCM_Espressif:ESP32-S3-DevKitC
Connections:
- net +5V: now also U3.7 (VIN); no longer U3.6 (VIN)
- net GND: now also U3.6 (GND), JP1.2 (B); no longer U3.7 (GND)
- net at J2.8 (Pin_8): now also JP1.1 (A)
Other:
- note added: "Mounting Holes"
- note removed: "MeanWell Power Supply Mounting Holes"
- note removed: "PCB-to-HUB75 Mounting Holes"
- note removed: "Speaker Mounting Holes"
